File: bspd.sch (KiCad schematic (older format))
At the start: 13 parts, among them U1 TI_NATIONAL_SEMICONDUCTOR_LMV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

Commit message: fix or gate
Parts:
- added C?: C, symbol Device:C
- added R?: R_US, symbol Device:R_US
- added U?: 74LVC1G32, symbol 74xGxx:74LVC1G32
Connections:
- net labels added: B_TH, C_TH, FAULT
- wire segments 39 -> 48
- no-connect marks 1 -> 2
Other:
- note added: "I HATE KICAD\n"
Changed lines of the file:
@@
 EESchema Schematic File Version 4
+LIBS:bspd-cache
 EELAYER 30 0
 EELAYER END
@@
 C_L
 $Comp
-L bspd:TI_NATIONAL_SEMICONDUCTOR_LMV7231SQE-NOPB U1
-U 1 1 5DF9F810
-P 4150 2050
-F 0 "U1" H 4774 1930 50  0000 C CNN
-F 1 "TI_NATIONAL_SEMICONDUCTOR_LMV7231SQE-NOPB" H 4150 2050 50  0001 L BNN
-F 2 "bspd:TI_NATIONAL_SEMICONDUCTOR_LMV7231SQE-NOPB_0" H 4150 2050 50  0001 L BNN
-F 3 "" H 4150 2050 50  0001 C CNN
-	1    4150 2050
-	1    0    0    -1
-$EndComp
-$Comp
 L power:GND #PWR015
 U 1 1 5DFA05A1
@@
 	1    0    0    -1
 $EndComp
-Wire Wire Line
-	5050 3650 5050 3750
-Connection ~ 5050 3750
-Wire Wire Line
-	5050 3750 5050 3950
-Connection ~ 5050 3950
-Wire Wire Line
-	5050 3950 5050 4050
-Connection ~ 5050 4050
-Wire Wire Line
-	5050 4050 5050 4100
 NoConn ~ 5050 3550
 $Comp
@@
 	3500 3450 3950 3450
 $Comp
+L 74xGxx:74LVC1G08 U?
+U 1 1 5DFC0A49
+P 5550 3300
+F 0 "U?" H 5525 3567 50  0000 C CNN
+F 1 "74LVC1G08" H 5525 3476 50  0000 C CNN
+F 2 "" H 5550 3300 50  0001 C CNN
+F 3 "http://www.ti.com/lit/sg/scyt129e/scyt129e.pdf" H 5550 3300 50  0001 C CNN
+	1    5550 3300
+	1    0    0    -1
+$EndComp
+Wire Wire Line
+	5050 3350 5250 3350
+Wire Wire Line
+	5050 3150 5150 3150
+Wire Wire Line
+	5150 3150 5150 3250
+Wire Wire Line
+	5150 3250 5250 3250
+Wire Wire Line
+	5050 2950 5750 2950
+Wire Wire Line
+	5750 2950 5750 2900
+Wire Wire Line
+	5750 2900 5900 2900
+Wire Wire Line
+	5050 2750 5550 2750
+Wire Wire Line
+	5550 2750 5550 2800
+Wire Wire Line
+	5550 2800 5900 2800
+Wire Wire Line
+	5600 2700 5900 2700
+$Comp
+L power:+5V #PWR?
+U 1 1 5DFA97B0
+P 5550 3200
+F 0 "#PWR?" H 5550 3050 50  0001 C CNN
+F 1 "+5V" H 5565 3373 50  0000 C CNN
+F 2 "" H 5550 3200 50  0001 C CNN
+F 3 "" H 5550 3200 50  0001 C CNN
+	1    5550 3200
+	1    0    0    -1
+$EndComp
+$Comp
+L power:GND #PWR?
+U 1 1 5DFAA4CA
+P 5550 3400
+F 0 "#PWR?" H 5550 3150 50  0001 C CNN
+F 1 "GND" H 5555 3227 50  0000 C CNN
+F 2 "" H 5550 3400 50  0001 C CNN
+F 3 "" H 5550 3400 50  0001 C CNN
+	1    5550 3400
+	1    0    0    -1
+$EndComp
+$Comp
+L Device:R_US R?
+U 1 1 5DFB1FA8
+P 5800 3450
+F 0 "R?" H 5868 3496 50  0000 L CNN
+F 1 "R_US" H 5868 3405 50  0000 L CNN
+F 2 "" V 5840 3440 50  0001 C CNN
+F 3 "~" H 5800 3450 50  0001 C CNN
+	1    5800 3450
+	1    0    0    -1
+$EndComp
+$Comp
+L Device:C C?
+U 1 1 5DFB2E43
+P 5800 3750
+F 0 "C?" H 5915 3796 50  0000 L CNN
+F 1 "C" H 5915 3705 50  0000 L CNN
+F 2 "" H 5838 3600 50  0001 C CNN
+F 3 "~" H 5800 3750 50  0001 C CNN
+	1    5800 3750
+	1    0    0    -1
+$EndComp
+$Comp
+L power:GND #PWR?
+U 1 1 5DFB3AE6
+P 5800 3900
+F 0 "#PWR?" H 5800 3650 50  0001 C CNN
+F 1 "GND" H 5805 3727 50  0000 C CNN
+F 2 "" H 5800 3900 50  0001 C CNN
+F 3 "" H 5800 3900 50  0001 C CNN
+	1    5800 3900
+	1    0    0    -1
+$EndComp
+Wire Wire Line
+	1350 2200 1150 2200
+Wire Wire Line
+	2300 2200 1900 2200
+Text Label 1200 2200 0    50   ~ 0
+B_TH
+Text Label 2000 2200 0    50   ~ 0
+C_TH
+Text Label 3500 3350 0    50   ~ 0
+C_TH
+Text Label 3500 3150 0    50   ~ 0
+B_TH
+$Comp
+L 74xGxx:74LVC1G32 U?
+U 1 1 5DFB7A4B
+P 5400 2400
+F 0 "U?" H 5375 2667 50  0000 C CNN
+F 1 "74LVC1G32" H 5375 2576 50  0000 C CNN
+F 2 "" H 5400 2400 50  0001 C CNN
+F 3 "http://www.ti.com/lit/sg/scyt129e/scyt129e.pdf" H 5400 2400 50  0001 C CNN
+	1    5400 2400
+	1    0    0    -1
+$EndComp
+Connection ~ 5050 3950
+Wire Wire Line
+	5050 3650 5050 3750
+Wire Wire Line
+	5050 3750 5050 3950
+Connection ~ 5050 3750
+Wire Wire Line
+	5050 3950 5050 4050
+Wire Wire Line
+	5050 4050 5050 4100
+Connection ~ 5050 4050
+$Comp
+L bspd:TI_NATIONAL_SEMICONDUCTOR_LMV7231SQE-NOPB U1
+U 1 1 5DF9F810
+P 4150 2050
+F 0 "U1" H 4774 1930 50  0000 C CNN
+F 1 "TI_NATIONAL_SEMICONDUCTOR_LMV7231SQE-NOPB" H 4150 2050 50  0001 L BNN
+F 2 "bspd:TI_NATIONAL_SEMICONDUCTOR_LMV7231SQE-NOPB_0" H 4150 2050 50  0001 L BNN
+F 3 "" H 4150 2050 50  0001 C CNN
+	1    4150 2050
+	1    0    0    -1
+$EndComp
+Wire Wire Line
+	5600 2400 5650 2400
+Wire Wire Line
+	5600 2400 5600 2700
+Wire Wire Line
+	5100 2450 5100 2550
+Wire Wire Line
+	5100 2550 5050 2550
+Wire Wire Line
+	5050 2350 5100 2350
+$Comp
+L power:GND #PWR?
+U 1 1 5DFC0D70
+P 5400 2500
+F 0 "#PWR?" H 5400 2250 50  0001 C CNN
+F 1 "GND" H 5405 2327 50  0000 C CNN
+F 2 "" H 5400 2500 50  0001 C CNN
+F 3 "" H 5400 2500 50  0001 C CNN
+	1    5400 2500
+	1    0    0    -1
+$EndComp
+$Comp
+L power:+5V #PWR?
+U 1 1 5DFC1509
+P 5400 2300
+F 0 "#PWR?" H 5400 2150 50  0001 C CNN
+F 1 "+5V" H 5415 2473 50  0000 C CNN
+F 2 "" H 5400 2300 50  0001 C CNN
+F 3 "" H 5400 2300 50  0001 C CNN
+	1    5400 2300
+	1    0    0    -1
+$EndComp
+Text Label 3500 2950 0    50   ~ 0
+C_H
+Text Label 3500 2750 0    50   ~ 0
+B_H
+Text Label 3500 2450 0    50   ~ 0
+B_L
+Text Label 3500 2650 0    50   ~ 0
+C_L
+NoConn ~ 7500 2900
+$Comp
+L power:+5V #PWR?
+U 1 1 5DFC3B5A
+P 7500 2650
+F 0 "#PWR?" H 7500 2500 50  0001 C CNN
+F 1 "+5V" H 7515 2823 50  0000 C CNN
+F 2 "" H 7500 2650 50  0001 C CNN
+F 3 "" H 7500 2650 50  0001 C CNN
+	1    7500 2650
+	1    0    0    -1
+$EndComp
+Wire Wire Line
+	7500 2650 7500 2700
+$Comp
+L power:GND #PWR?
+U 1 1 5DFC51B6
+P 7500 3000
+F 0 "#PWR?" H 7500 2750 50  0001 C CNN
+F 1 "GND" H 7505 2827 50  0000 C CNN
+F 2 "" H 7500 3000 50  0001 C CNN
+F 3 "" H 7500 3000 50  0001 C CNN
+	1    7500 3000
+	1    0    0    -1
+$EndComp
+Wire Wire Line
+	8550 2800 7500 2800
+Text Label 8000 2800 0    50   ~ 0
+FAULT
+$Comp
 L bspd:MC100EP01DTG U?
 U 1 1 5DFBF5C3
@@
 	1    0    0    -1
 $EndComp
-$Comp
-L 74xGxx:74LVC1G08 U?
-U 1 1 5DFC0A49
-P 5550 3300
-F 0 "U?" H 5525 3567 50  0000 C CNN
-F 1 "74LVC1G08" H 5525 3476 50  0000 C CNN
-F 2 "" H 5550 3300 50  0001 C CNN
-F 3 "http://www.ti.com/lit/sg/scyt129e/scyt129e.pdf" H 5550 3300 50  0001 C CNN
-	1    5550 3300
-	1    0    0    -1
-$EndComp
-Wire Wire Line
-	5050 3350 5250 3350
-Wire Wire Line
-	5050 3150 5150 3150
-Wire Wire Line
-	5150 3150 5150 3250
-Wire Wire Line
-	5150 3250 5250 3250
-Wire Wire Line
-	5800 3300 5800 3000
-Wire Wire Line
-	5800 3000 5900 3000
-Wire Wire Line
-	5050 2950 5750 2950
-Wire Wire Line
-	5750 2950 5750 2900
-Wire Wire Line
-	5750 2900 5900 2900
-Wire Wire Line
-	5050 2750 5550 2750
-Wire Wire Line
-	5550 2750 5550 2800
-Wire Wire Line
-	5550 2800 5900 2800
-Wire Wire Line
-	5050 2550 5600 2550
-Wire Wire Line
-	5600 2550 5600 2700
-Wire Wire Line
-	5600 2700 5900 2700
+Wire Wire Line
+	5800 3600 6050 3600
+Wire Wire Line
+	6050 3600 6050 3150
+Wire Wire Line
+	6050 3150 5900 3150
+Wire Wire Line
+	5900 3150 5900 3000
+Connection ~ 5800 3600
+Text Notes 2500 5600 0    50   ~ 0
+I HATE KICAD\n
 $EndSCHEMATC
